Commit message: lidar,odom working

File: rover_ws/install/gazebo/share/gazebo/model/rover.xacro (robot description, xacro)
@@ -2,7 +2,4 @@
 <robot xmlns:xacro="http://www.ros.org/wiki/xacro" name= "rover">
 <xacro:include filename="$(find gazebo)/model/rover.gazebo"/>
-<xacro:property name = "body_link_y_dim" value = "1"/>
-<xacro:property name = "wheel_link_length" value = "0.05"/>
-<xacro:property name = "wheel_link_radius" value = "0.15"/>
 <material name = "black">
     <color rgba = " 0 0 0 1"/>
@@ -51,5 +48,5 @@
     <origin xyz = "0.275 0.45 0" rpy = "0 0 0" />
     <axis xyz ="1 0 0"/>
-    <limit effort = "1000" velocity = "1000"/>
+    <limit effort = "10" velocity = "5"/>
     <dynamics damping = "1.0" friction = "1.0"/>
 </joint>
@@ -70,5 +67,5 @@
     <inertial>
          <origin xyz = " 0 0 0" rpy = "0 1.57 0"/>
-        <mass value= "0.25"/>
+        <mass value= "0.5"/>
         <inertia ixx = "100" ixy = "0" ixz = "0" iyy = "100" izz = "100" iyz = "0"/>
     </inertial>
@@ -79,5 +76,5 @@
     <origin xyz = "-0.275 0.45 0" rpy = "0 0 0" />
     <axis xyz ="1 0 0"/>
-    <limit effort = "1000" velocity = "1000"/>
+    <limit effort = "10" velocity = "5"/>
     <dynamics damping = "1.0" friction = "1.0"/>
 </joint>
@@ -98,5 +95,5 @@
     <inertial>
          <origin xyz = " 0 0 0" rpy = "0 1.57 0"/>
-        <mass value= "0.25"/>
+        <mass value= "0.5"/>
         <inertia ixx = "100" ixy = "0" ixz = "0" iyy = "100" izz = "100" iyz = "0"/>
     </inertial>
@@ -107,5 +104,5 @@
     <origin xyz = "0.275 -0.45 0" rpy = "0 0 0" />
     <axis xyz ="1 0 0"/>
-    <limit effort = "1000" velocity = "1000"/>
+    <limit effort = "10" velocity = "5"/>
     <dynamics damping = "1.0" friction = "1.0"/>
 </joint>
@@ -126,5 +123,5 @@
     <inertial>
          <origin xyz = " 0 0 0" rpy = "0 1.57 0"/>
-        <mass value= "0.25"/>
+        <mass value= "0.5"/>
         <inertia ixx = "100" ixy = "0" ixz = "0" iyy = "100" izz = "100" iyz = "0"/>
     </inertial>
@@ -135,5 +132,5 @@
     <origin xyz = "-0.275 -0.45 0" rpy = "0 0 0" />
     <axis xyz ="1 0 0"/>
-    <limit effort = "1000" velocity = "1000"/>
+    <limit effort = "10" velocity = "5"/>
     <dynamics damping = "1.0" friction = "1.0"/>
 </joint>
@@ -154,5 +151,5 @@
     <inertial>
          <origin xyz = " 0 0 0" rpy = "0 1.57 0"/>
-        <mass value= "0.25"/>
+        <mass value= "0.5"/>
         <inertia ixx = "100" ixy = "0" ixz = "0" iyy = "100" izz = "100" iyz = "0"/>
     </inertial>
@@ -163,45 +160,56 @@
     <origin xyz = "0 0.45 0.275" rpy = "0 0 0" />
 </joint>
-    <link name = "lidar_link">
-        <sensor type="lidar" name="lidar">
-            <laser>
-                <scan>
-                    <horizontal>
-                        <samples>1081</samples>
-                        <resolution>1.0</resolution>
-                    </horizontal>
-                </scan>
-                <range>
-                    <min>0.2</min>
-                    <max>30.0</max>
-                </range>
-            </laser>
-        </sensor>
-       <plugin name="lidar_plugin" filename="libgazebo_ros_laser.so">
-    <ros>
-        <namespace>lidar</namespace>
-        <remapping>scan:=/lidar/scan</remapping>
-        <param name="frame_id" value="lidar_link"/>
-    </ros>
-</plugin>
-        <visual>
-            <geometry>
-                <box size = " 0.1 0.1 0.05 "/>
-            </geometry>
-            <origin xyz = " 0 0 0" rpy = "0 0 0"/>
-            <material name = "red"/>
-        </visual>
-     <collision>
-            <geometry>
-                <box size = " 0.1 0.1 0.05 "/>
-            </geometry>
-            <origin xyz = " 0 0 0" rpy = "0 0 0"/>
-    </collision>
-    <inertial>
-         <origin xyz = " 0 0 0" rpy = "0 0 0"/>
-        <mass value= "0.25"/>
-        <inertia ixx = "100" ixy = "0" ixz = "0" iyy = "100" izz = "100" iyz = "0"/>
-    </inertial>
-    </link>
+ <link name="lidar_link">
+    <visual>
+      <geometry>
+        <cylinder radius="0.05" length="0.1"/>
+      </geometry>
+      <material name="green"/>
+    </visual>
+    <collision>
+      <geometry>
+        <cylinder radius="0.05" length="0.1"/>
+      </geometry>
+    </collision>
+    <inertial>
+      <mass value="0.5"/>
+      <inertia ixx="0.01" ixy="0" ixz="0" iyy="0.01" iyz="0" izz="0.01"/>
+    </inertial>
+  </link>
+  <!-- Gazebo Plugin for Lidar -->
+  <gazebo reference="lidar_link">
+    <sensor name="lidar_sensor" type="ray">
+      <pose>0 0 0 0 0 0</pose>
+      <visualize>true</visualize>
+      <update_rate>10</update_rate>
+      <ray>
+        <scan>
+          <horizontal>
+            <samples>360</samples>
+            <resolution>1</resolution>
+            <min_angle>-3.14159</min_angle>
+            <max_angle>3.14159</max_angle>
+          </horizontal>
+        </scan>
+        <range>
+          <min>0.1</min>
+          <max>10.0</max>
+          <resolution>0.01</resolution>
+        </range>
+        <noise>
+          <type>gaussian</type>
+          <mean>0.0</mean>
+          <stddev>0.01</stddev>
+        </noise>
+      </ray>
+      <plugin name="lidar_plugin" filename="libgazebo_ros_ray_sensor.so">
+        <ros>
+          <namespace>lidar</namespace>
+          <remapping>~/out:=scan</remapping>
+        </ros>
+        <frame_name>lidar_link</frame_name>
+      </plugin>
+    </sensor>
+  </gazebo>
 <joint name = "imu_joint" type = "fixed">
     <parent link = "base_link"/>
@@ -209,158 +217,157 @@
     <origin xyz = "0 -0.45 0.275" rpy = "0 0 0" />
 </joint>
-    <link name = "imu_link">
-         <sensor type="imu" name="imu">
-            <imu>
-                <update_rate>100.0</update_rate>
-                <raw>true</raw>
-                <frame_id>imu_link</frame_id>
-            </imu>
-        </sensor>
-        <plugin name="imu_plugin" filename="libgazebo_ros_imu.so">
-    <ros>
-        <namespace>imu</namespace>
-        <remapping>imu/data:=/imu/data</remapping>
-        <param name="frame_id" value="imu_link"/>
-    </ros>
-</plugin>
-        <visual>
-            <geometry>
-                <box size = " 0.1 0.1 0.05 "/>
-            </geometry>
-            <origin xyz = " 0 0 0" rpy = "0 0 0"/>
-            <material name = "blue"/>
-        </visual>
-    <collision>
-            <geometry>
-                <box size = " 0.1 0.1 0.05 "/>
-            </geometry>
-            <origin xyz = " 0 0 0" rpy = "0 0 0"/>
-    </collision>
-    <inertial>
-         <origin xyz = " 0 0 0" rpy = "0 0 0"/>
-        <mass value= "0.25"/>
-        <inertia ixx = "100" ixy = "0" ixz = "0" iyy = "100" izz = "100" iyz = "0"/>
-    </inertial>
-    </link>
+  <!-- IMU Link -->
+  <link name="imu_link">
+    <visual>
+      <geometry>
+        <cylinder radius="0.05" length="0.04"/>
+      </geometry>
+       <origin xyz="0 0 0" rpy="0 0 0"/>
+      <material name="black">
+        <color rgba="0 1 0 1"/>
+      </material>
+    </visual>
+    <collision>
+      <geometry>
+        <cylinder radius="0.05" length="0.04"/>
+      </geometry>
+    </collision>
+  <gazebo reference="imu_link">
+    <sensor name="imu_sensor" type="imu">
+      <always_on>true</always_on>
+      <update_rate>10.0</update_rate>
+      <plugin name="imu_controller" filename="libgazebo_ros_imu_sensor.so">
+        <ros>
+          <remapping>imu_controller/out:=imu</remapping>
+        </ros>
+        <frame_name>imu_link</frame_name>
+      </plugin>
+    </sensor>
+    <material>Gazebo/Grey</material>
+  </gazebo>
+  </link>
     <!-- GPS Sensor -->
-    <link name="gps_link">
-        <plugin name="gps_plugin" filename="libgazebo_ros_gps.so">
-    <ros>
-        <namespace>gps</namespace>
-        <remapping>fix:=/gps/fix</remapping>
-        <remapping>velocity:=/gps/vel</remapping>
-        <param name="frame_id" value="gps_link"/>
-    </ros>
-</plugin>
-        <visual>
-            <geometry>
-                <box size = " 0.1 0.1 0.05 "/>
-            </geometry>
-            <origin xyz = " 0 0 0" rpy = "0 0 0"/>
-            <material name = "red"/>
-        </visual>
-     <collision>
-            <geometry>
-                <box size = " 0.1 0.1 0.05 "/>
-            </geometry>
-            <origin xyz = " 0 0 0" rpy = "0 0 0"/>
-    </collision>
-    <inertial>
-         <origin xyz = " 0 0 0" rpy = "0 0 0"/>
-        <mass value= "0.25"/>
-        <inertia ixx = "100" ixy = "0" ixz = "0" iyy = "100" izz = "100" iyz = "0"/>
-    </inertial>
-        <sensor type="gps" name="gps">
-            <gps>
-                <update_rate>1.0</update_rate>
-                <frame_id>gps_link</frame_id>
-            </gps>
-        </sensor>
-    </link>
+  <link name="gps_link">
+    <visual>
+      <geometry>
+        <cylinder radius="0.05" length="0.04"/>
+      </geometry>
+      <origin xyz="0 0 0" rpy="0 0 0"/>
+      <material name="black">
+        <color rgba="0 1 0 1"/>
+      </material>
+    </visual>
+    <collision>
+      <geometry>
+        <cylinder radius="0.05" length="0.04"/>
+      </geometry>
+    </collision>
+    </link>
+<gazebo reference="gps_link">
+    <sensor name="gps_sensor" type="gps">
+        <always_on>true</always_on>
+        <update_rate>1.0</update_rate>
+        <plugin name="gps_controller" filename="libgazebo_ros_gps_sensor.so">
+            <ros>
+                <remapping>gps_controller/out:=gps</remapping>
+            </ros>
+            <frame_name>gps_link</frame_name>
+        </plugin>
+    </sensor>
+    <material>Gazebo/Grey</material>
+</gazebo>
 <joint name = "gps_joint" type = "fixed">
     <parent link = "base_link"/>
     <child link = "gps_link"/>
-    <origin xyz = "0 0 0.275" rpy = "0 0 0" />
+    <origin xyz = "-0.2 0 0.275" rpy = "0 0 0" />
 </joint>
 <joint name = "camera_joint" type = "fixed">
     <parent link = "base_link"/>
-    <child link = "stereo_camera_link"/>
-    <origin xyz = "0.25 0 0.275" rpy = "0 0 0" />
-</joint>
-    <!-- Stereo Camera Sensor Definition -->
-    <link name="stereo_camera_link">
-          <visual>
-            <geometry>
-                <box size = " 0.1 0.1 0.05 "/>
-            </geometry>
-            <origin xyz = " 0 0 0" rpy = "0 0 0"/>
-            <material name = "red"/>
-        </visual>
-     <collision>
-            <geometry>
-                <box size = " 0.1 0.1 0.05 "/>
-            </geometry>
-            <origin xyz = " 0 0 0" rpy = "0 0 0"/>
-    </collision>
-    <inertial>
-         <origin xyz = " 0 0 0" rpy = "0 0 0"/>
-        <mass value= "0.25"/>
-        <inertia ixx = "100" ixy = "0" ixz = "0" iyy = "100" izz = "100" iyz = "0"/>
-    </inertial>
-        <sensor type="camera" name="left_camera">
-            <camera>
+    <child link = "camera_link"/>
+    <origin xyz = "0.2 0 0.275" rpy = "0 0 0" />
+</joint>
+    <link name="camera_link">
+        <visual>
+            <geometry>
+            <box size="0.05 0.05 0.05"/>
+            </geometry>
+            <material name="white"/>
+        </visual>
+         <gazebo reference="camera_link">
+        <sensor type="depth" name="my_camera">
+            <update_rate>20</update_rate>
+            <visualize>true</visualize>
+            <camera name="cam">
                 <horizontal_fov>1.3962634</horizontal_fov>
                 <image>
                     <width>640</width>
                     <height>480</height>
-                    <format>R8G8B8</format>
+                    <format>R8B8G8</format>
                 </image>
-                <update_rate>30.0</update_rate>
-                <camera_info>
-                    <intrinsics>
-                        <fx>500.0</fx>
-                        <fy>500.0</fy>
-                        <cx>320.0</cx>
-                        <cy>240.0</cy>
-                    </intrinsics>
-                </camera_info>
+                <clip>
+                    <near>0.02</near>
+                    <far>300</far>
+                </clip>
+                <noise>
+                    <type>gaussian</type>
+                    <mean>0.0</mean>
+                    <stddev>0.007</stddev>
+                </noise>
             </camera>
+            <plugin name="camera_controller" filename="libgazebo_ros_camera.so">
+                <frame_name>camera_link_optical</frame_name>
+                <min_depth>0.1</min_depth>
+                <max_depth>500</max_depth>
+            </plugin>
         </sensor>
-        <plugin name="stereo_camera_plugin" filename="libgazebo_ros_stereo_camera.so">
-    <ros>
-        <namespace>stereo_camera</namespace>
-        <remapping>left/image_raw:=/stereo_camera/left/image_raw</remapping>
-        <remapping>right/image_raw:=/stereo_camera/right/image_raw</remapping>
-        <remapping>left/camera_info:=/stereo_camera/left/camera_info</remapping>
-        <remapping>right/camera_info:=/stereo_camera/right/camera_info</remapping>
-    </ros>
-    <left_camera>
-        <name>left_camera</name>
-        <update_rate>30.0</update_rate>
-    </left_camera>
-    <right_camera>
-        <name>right_camera</name>
-        <update_rate>30.0</update_rate>
-    </right_camera>
-</plugin>
-        <sensor type="camera" name="right_camera">
-            <camera>
-                <horizontal_fov>1.3962634</horizontal_fov>
-                <image>
-                    <width>640</width>
-                    <height>480</height>
-                    <format>R8G8B8</format>
-                </image>
-                <update_rate>30.0</update_rate>
-                <camera_info>
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
Commit message: Final working rover

File: rover_ws/install/gazebo/share/gazebo/model/rover.xacro (robot description, xacro)
@@ -326,5 +326,5 @@
         <parent link="base_link"/>
         <child link="stereo_link"/>
-        <origin xyz="0.3 0 0.1" rpy="-1.57 -1.57 -1.57"/>
+        <origin xyz="0.2 0.2 0.275" rpy="0 0 0"/>
     </joint>
     <link name="stereo_link">
